File: hardware_design/prototyping_buttons_daughterboard/prototyping_backplane/prototyping_backplane.sch (KiCad schematic (older format))
At the start: 11 parts, among them J1 BOOSTER_LEFT, J2 BOOSTER_RIGHT, J3 EXP_SPI, SW1 SW_DIP_x01 CUT LEADS, SW2 SW_DIP_x02

Commit message: Increment to dev version, add basic hardware functionality for audio, add simple sound test
Parts:
- J3: footprint Connector_PinHeader_2.00mm:PinHeader_1x04_P2.00mm_Horizontal -> Connector_PinHeader_2.00mm:PinHeader_1x06_P2.00mm_Horizontal; symbol Connector:Conn_01x04_Female -> Connector:Conn_01x06_Female
Connections:
- net at BT1.2 (-), J2.2 (Pin_2), SW2.3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: now also J3.6 (Pin_6)
- net at J1.1 (Pin_1), SW1.2: now also J3.1 (Pin_1)
- net at J1.13 (Pin_13): now also J3.3 (Pin_3); no longer J3.4 (Pin_4)
- net at J1.20 (Pin_20): now also J3.2 (Pin_2); no longer J3.3 (Pin_3)
- net at J2.10 (Pin_10): no longer J3.1 (Pin_1)
- net at J2.12 (Pin_12): now also J3.4 (Pin_4); no longer J3.2 (Pin_2)
- net at J2.14 (Pin_14): now also J3.5 (Pin_5)
- no-connect marks 13 -> 12
Changed lines of the file:
@@
 NoConn ~ 8900 4550
 NoConn ~ 8900 4650
-NoConn ~ 8900 4950
-NoConn ~ 8900 5050
-NoConn ~ 8900 5150
 NoConn ~ 4800 4600
 NoConn ~ 4800 5100
@@
 Wire Wire Line
 	4800 4900 4400 4900
-Wire Wire Line
-	4400 4900 4400 5550
-Wire Wire Line
-	4400 5550 4250 5550
-Wire Wire Line
-	5300 5200 5300 5650
-Wire Wire Line
-	5300 5650 4250 5650
-Wire Wire Line
-	9550 6100 4250 6100
-Wire Wire Line
-	4250 6100 4250 5850
-Wire Wire Line
-	4250 5750 4450 5750
-Wire Wire Line
-	4450 5750 4450 5850
-Wire Wire Line
-	4450 5850 9300 5850
-Wire Wire Line
-	9300 5850 9300 4850
-Wire Wire Line
-	8900 4850 9300 4850
-Wire Wire Line
-	8900 4750 9550 4750
-Wire Wire Line
-	9550 4750 9550 6100
 $Comp
 L Switch:SW_DIP_x02 SW2
@@
 Wire Wire Line
 	9550 3750 9550 4350
+Wire Wire Line
+	5850 2200 9550 2200
+$Comp
+L Connector:Conn_01x06_Female J3
+U 1 1 6127399A
+P 3850 5650
+F 0 "J3" H 3878 5626 50  0000 L CNN
+F 1 "EXP_SPI" H 3878 5535 50  0000 L CNN
+F 2 "Connector_PinHeader_2.00mm:PinHeader_1x06_P2.00mm_Horizontal" H 3850 5650 50  0001 C CNN
+F 3 "~" H 3850 5650 50  0001 C CNN
+	1    3850 5650
+	-1   0    0    -1
+$EndComp
+Wire Wire Line
+	5450 5700 5450 5100
+Wire Wire Line
+	5450 5100 5300 5100
+Wire Wire Line
+	5500 5000 5300 5000
+Wire Wire Line
+	5500 5000 5500 5350
+Wire Wire Line
+	5300 4400 6600 4400
+Wire Wire Line
+	8400 4600 8400 4650
+Wire Wire Line
+	6600 5350 6600 4400
+Wire Wire Line
+	6450 5350 6600 5350
+Connection ~ 6600 5350
+Wire Wire Line
+	6600 5350 7050 5350
+Wire Wire Line
+	8400 4600 7450 4600
+Wire Wire Line
+	7450 4600 7450 4400
+Wire Wire Line
+	7450 4400 7250 4400
+Connection ~ 6600 4400
+Wire Wire Line
+	6600 4400 7150 4400
+Wire Wire Line
+	4350 4300 4050 4300
+Wire Wire Line
+	4050 4300 4050 5450
+Connection ~ 4350 4300
+Wire Wire Line
+	4050 5950 4150 5950
+Wire Wire Line
+	4150 5950 4150 6250
+Wire Wire Line
+	4150 6250 9850 6250
+Wire Wire Line
+	9850 6250 9850 2200
+Wire Wire Line
+	9850 2200 9550 2200
+Connection ~ 9550 2200
+Wire Wire Line
+	4400 5650 4050 5650
+Wire Wire Line
+	4400 4900 4400 5650
+Wire Wire Line
+	5300 5200 5300 5550
+Wire Wire Line
+	5300 5550 4050 5550
+NoConn ~ 4400 5550
 $Comp
 L Connector_Generic:Conn_02x10_Odd_Even J2
@@
 $EndComp
 Wire Wire Line
-	5850 2200 9550 2200
-$Comp
-L Connector:Conn_01x04_Female J3
-U 1 1 6127399A
-P 4050 5750
-F 0 "J3" H 4078 5726 50  0000 L CNN
-F 1 "EXP_SPI" H 4078 5635 50  0000 L CNN
-F 2 "Connector_PinHeader_2.00mm:PinHeader_1x04_P2.00mm_Horizontal" H 4050 5750 50  0001 C CNN
-F 3 "~" H 4050 5750 50  0001 C CNN
-	1    4050 5750
-	-1   0    0    1
-$EndComp
-Wire Wire Line
-	5450 5700 5450 5100
-Wire Wire Line
-	5450 5100 5300 5100
-Wire Wire Line
-	5500 5000 5300 5000
-Wire Wire Line
-	5500 5000 5500 5350
-Wire Wire Line
-	5300 4400 6600 4400
-Wire Wire Line
-	8400 4600 8400 4650
-Wire Wire Line
-	6600 5350 6600 4400
-Wire Wire Line
-	6450 5350 6600 5350
-Connection ~ 6600 5350
-Wire Wire Line
-	6600 5350 7050 5350
-Wire Wire Line
-	8400 4600 7450 4600
-Wire Wire Line
-	7450 4600 7450 4400
-Wire Wire Line
-	7450 4400 7250 4400
-Connection ~ 6600 4400
-Wire Wire Line
-	6600 4400 7150 4400
+	9000 4950 8900 4950
+Wire Wire Line
+	9100 5850 9100 4850
+Wire Wire Line
+	9100 4850 8900 4850
+Wire Wire Line
+	9100 5850 4700 5850
+Wire Wire Line
+	4700 5850 4700 5750
+Wire Wire Line
+	4700 5750 4050 5750
+Wire Wire Line
+	9000 5950 4450 5950
+Wire Wire Line
+	4450 5950 4450 5850
+Wire Wire Line
+	4450 5850 4050 5850
+Wire Wire Line
+	9000 4950 9000 5950
+NoConn ~ 9000 5850
 $EndSCHEMATC
