File: hardware_design/prototyping_buttons_daughterboard/prototyping_buttons_daughterboard.kicad_pcb (KiCad board)
At the start: 2 copper layers, 80 x 32.5 mm, 10 parts, among them J1 Conn_02x10_Counter_Clockwise, J2 Conn_02x10_Counter_Clockwise

Commit message: catchup of documentation-related work
Parts:
- J1, J2: moved to B.Cu
- moved J2 2.55 mm to (127.0, 53.3), turned to 180 degrees
- moved J1 2.54 mm to (83.8, 53.3), turned to 180 degrees
Connections:
- C1 pad 1: Net-(C1-Pad1) -> Net-(J1-Pad4)
- C1 pad 2: Net-(C1-Pad2) -> Net-(J1-Pad7)
- C2 pad 2: Net-(C1-Pad1) -> Net-(J1-Pad4)
- J1 pad 1: Net-(J1-Pad1) -> unconnected-(J1-Pad1)
- J1 pad 10: Net-(J1-Pad10) -> unconnected-(J1-Pad10)
- J1 pad 11: Net-(J1-Pad11) -> unconnected-(J1-Pad11)
- J1 pad 12: Net-(J1-Pad12) -> unconnected-(J1-Pad12)
- J1 pad 13: Net-(J1-Pad13) -> unconnected-(J1-Pad13)
- J1 pad 14: Net-(J1-Pad14) -> unconnected-(J1-Pad14)
- J1 pad 15: Net-(J1-Pad15) -> unconnected-(J1-Pad15)
- J1 pad 16: Net-(J1-Pad16) -> unconnected-(J1-Pad16)
- J1 pad 17: Net-(J1-Pad17) -> Net-(C2-Pad1)
- J1 pad 18: Net-(C2-Pad1) -> unconnected-(J1-Pad18)
- J1 pad 19: Net-(J1-Pad19) -> unconnected-(J1-Pad19)
- J1 pad 2: Net-(J1-Pad2) -> unconnected-(J1-Pad2)
- J1 pad 20: Net-(J1-Pad20) -> unconnected-(J1-Pad20)
- J1 pad 3: Net-(C1-Pad1) -> unconnected-(J1-Pad3)
- J1 pad 5: Net-(J1-Pad5) -> unconnected-(J1-Pad5)
- J1 pad 6: Net-(J1-Pad6) -> unconnected-(J1-Pad6)
- J1 pad 8: Net-(C1-Pad2) -> unconnected-(J1-Pad8)
- J1 pad 9: Net-(J1-Pad9) -> unconnected-(J1-Pad9)
- J2 pad 1: Net-(C3-Pad1) -> unconnected-(J2-Pad1)
- J2 pad 10: Net-(J2-Pad10) -> unconnected-(J2-Pad10)
- J2 pad 11: Net-(J2-Pad11) -> unconnected-(J2-Pad11)
- J2 pad 12: Net-(J2-Pad12) -> unconnected-(J2-Pad12)
- J2 pad 13: Net-(J2-Pad13) -> unconnected-(J2-Pad13)
- J2 pad 14: Net-(J2-Pad14) -> unconnected-(J2-Pad14)
- J2 pad 15: Net-(C4-Pad1) -> unconnected-(J2-Pad15)
- J2 pad 16: Net-(J2-Pad16) -> Net-(C4-Pad1)
- J2 pad 17: Net-(J2-Pad17) -> unconnected-(J2-Pad17)
- J2 pad 18: Net-(J2-Pad18) -> unconnected-(J2-Pad18)
- J2 pad 19: Net-(J2-Pad19) -> unconnected-(J2-Pad19)
- J2 pad 2: Net-(J2-Pad2) -> Net-(C3-Pad1)
- J2 pad 20: Net-(J2-Pad20) -> unconnected-(J2-Pad20)
- J2 pad 3: Net-(C3-Pad2) -> unconnected-(J2-Pad3)
- J2 pad 4: Net-(J2-Pad4) -> Net-(C3-Pad2)
- J2 pad 5: Net-(J2-Pad5) -> unconnected-(J2-Pad5)
- J2 pad 6: Net-(J2-Pad6) -> unconnected-(J2-Pad6)
- J2 pad 7: Net-(J2-Pad7) -> unconnected-(J2-Pad7)
- J2 pad 8: Net-(J2-Pad8) -> unconnected-(J2-Pad8)
- J2 pad 9: Net-(J2-Pad9) -> unconnected-(J2-Pad9)
- SW-A1 pad 1: Net-(C1-Pad1) -> Net-(J1-Pad4)
- SW-A1 pad 2: Net-(C1-Pad2) -> Net-(J1-Pad7)
- SW-B1 pad 1: Net-(C1-Pad1) -> Net-(J1-Pad4)
Routing:
- net Net-(J1-Pad4): track 0.00 -> 81.2 mm
- net Net-(C1-Pad1): track 81.2 -> 0.00 mm
- net Net-(J1-Pad7): track 0.00 -> 19.0 mm
- net Net-(C1-Pad2): track 19.0 -> 0.00 mm
Other:
- net class Default removed
