File: hardware_design/prototyping_backplane/prototyping_backplane.kicad_pcb (KiCad board)
At the start: 2 copper layers, 57.6 x 83.8 mm, 25 parts, among them J1 BOOSTER_LEFT, J2 BOOSTER_RIGHT, J3 EXP_SPI, J4 EXP_LCD_CS, SW1 SW_DIP_x03, U1 TPS60204DGS

Commit message: Update schematics for revision D to close issue 35. PCB not complete, see release notes.
Connections:
- D1 pad 1: GROUND -> Net-(D1-Pad1)
- D1 pad 2: Net-(D1-Pad2) -> GROUND
- D2 pad 1: GROUND -> Net-(D2-Pad1)
- D2 pad 2: Net-(D2-Pad2) -> GROUND
- R1 pad 1: Net-(D2-Pad2) -> Net-(D2-Pad1)
- R2 pad 2: Net-(D1-Pad2) -> Net-(D1-Pad1)
Routing:
- net GROUND: track 249.1 -> 415.1 mm
- net 3_3V: track 106.6 -> 0.00 mm
- net SUPPLY: track 59.5 -> 0.00 mm
- net Net-(D2-Pad2): track 12.8 -> 0.00 mm
- net Net-(D2-Pad1): track 0.00 -> 12.8 mm
- net Net-(D1-Pad2): track 11.2 -> 0.00 mm
- net Net-(D1-Pad1): track 0.00 -> 11.2 mm

Commit message: update/finalize revD backplanes
Parts:
- added Q1: 2N2222A, Package_TO_SOT_THT:TO-92, B.Cu at (193.7, 61.9)
- LS1: value Device Buzzer -> AST-02308MR-R; footprint Buzzer_Beeper:Buzzer_12x9.5RM7.6 -> footprints:Buzzer_D20mm_H7mm_P10mm
- moved ? 92.7 mm to (45.6, 9.58)
- moved LS1 9.34 mm to (158.7, 62.9), turned to 0 degrees
- moved G*** 7.35 mm to (202.7, 65.9), turned to 90 degrees
Connections:
- LS1 pad 1: BUZZER -> Net-(Q1-E)
Routing:
- net GROUND: track 415.1 -> 245.6 mm
- net 3_3V: track 0.00 -> 122.6 mm
- net SUPPLY: track 0.00 -> 59.5 mm
- net Net-(Q1-E): track 0.00 -> 41.4 mm
- net BUZZER: track 71.0 -> 34.3 mm
- net MOSI: track 49.9 -> 52.5 mm
- net MISO: track 51.9 -> 53.0 mm
- net Net-(D2-K): track 12.8 -> 11.7 mm
- net Net-(D1-K): track 11.2 -> 10.2 mm
